File: efm8-v2-slim-no-pullups/tetrabyte-slim.sch (EAGLE design)
At the start: 18 parts, among them J1 TYPE-C-31-M-12, U1 EFM8UB20F64G-B-QFP48

Commit message: add bootload switch
Parts:
- added SW1: KMR211NGLFS, adafruit:SPST_TACT-KMR2
Connections:
- net BTLD: now also SW1.P
- net GND: now also SW1.S, SW1.S1
Changed lines of the file:
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@@
 <part name="S4" library="switch-dil" deviceset="DS08" device=""/>
 <part name="SUPPLY1" library="supply2" deviceset="GND" device=""/>
+<part name="GND7" library="supply1" deviceset="GND" device=""/>
+<part name="SW1" library="adafruit" deviceset="SPST_TACT" device="-KMR2" value="KMR211NGLFS "/>
 </parts>
 <sheets>
@@
 <instance part="S4" gate="A" x="68.58" y="106.68" rot="MR270"/>
 <instance part="SUPPLY1" gate="GND" x="55.88" y="91.44" rot="MR0"/>
+<instance part="GND7" gate="1" x="289.56" y="104.14" rot="MR0"/>
+<instance part="SW1" gate="G$1" x="294.64" y="111.76" smashed="yes" rot="MR270">
+<attribute name="NAME" x="294.64" y="106.68" size="1.778" layer="95"/>
+<attribute name="VALUE" x="294.64" y="104.14" size="1.778" layer="96"/>
+</instance>
 </instances>
 <busses>
@@
 <junction x="55.88" y="154.94"/>
 </segment>
+<segment>
+<wire x1="289.56" y1="106.68" x2="289.56" y2="109.22" width="0.1524" layer="91"/>
+<wire x1="289.56" y1="111.76" x2="289.56" y2="109.22" width="0.1524" layer="91"/>
+<junction x="289.56" y="109.22"/>
+<pinref part="GND7" gate="1" pin="GND"/>
+<pinref part="SW1" gate="G$1" pin="S"/>
+<pinref part="SW1" gate="G$1" pin="S1"/>
+</segment>
 </net>
 <net name="+5V" class="0">
@@
 </segment>
 </net>
-<net name="BTLD" class="0">
-<segment>
-<pinref part="U1" gate="G$1" pin="P3.7"/>
-<wire x1="350.52" y1="144.78" x2="350.52" y2="121.92" width="0.1524" layer="91"/>
-<label x="350.52" y="121.92" size="1.778" layer="95" rot="R90"/>
-</segment>
-</net>
 <net name="S3-2" class="0">
 <segment>
@@
 </segment>
 </net>
+<net name="BTLD" class="0">
+<segment>
+<pinref part="SW1" gate="G$1" pin="P"/>
+<pinref part="U1" gate="G$1" pin="P3.7"/>
+<wire x1="350.52" y1="144.78" x2="350.52" y2="111.76" width="0.1524" layer="91"/>
+<label x="350.52" y="121.92" size="1.778" layer="95" rot="R90"/>
+<wire x1="299.72" y1="111.76" x2="350.52" y2="111.76" width="0.1524" layer="91"/>
+</segment>
+</net>
